File: rowan/rowan.kicad_pcb (KiCad board)
At the start: 2 copper layers, 131.8 x 57.6 mm, 115 parts, among them J1 Conn_01x02, J10 Conn_01x03, J11 Conn_02x05_Odd_Even, J12 Conn_01x04, J13 Conn_01x03, J14 Conn_01x03, J15 Conn_01x03, J16 Conn_01x08, J17 Conn_01x08, J2 USB_C_Receptacle_USB2.0_16P, J3 AudioJack2, J4 AudioJack2, J5 AudioJack2, J6 AudioJack2, J7 AudioJack2, J8 AudioJack2, J9 Conn_01x03, SW1 SW_Push, U1 DAC7554, U10 NCP1117-5.0_SOT223, U2 NCP1117-3.3_SOT223, U3 MCP6002-xMS, U4 MCP6002-xMS, U5 W25Q32JVSS, U6 RP2040, U7 74AHCT1G125, U8 74AHCT1G125, U9 LM4040LP-5, Y2 Crystal_GND2

Commit message: Updating the Rowan PCB for production run
Declares version 1.1, and sets the year
Other:
- board text added: "Rowan 1.1 (Production 1) Tom Carlson 2024-2025 hello@divergentwaves.co.uk"
- board text removed: "Bottom board to top board: Trig A Trig B Earth Unquant A Chro A Earth Unquant B Chro B Earth LED driver +5v Earth"
- board text removed: "LED centerline (Top)"
- board text removed: "Rowan 1.0 (Prototype 1) Tom Carlson 2024 hello@divergentwaves.co.uk"
- board text removed: "TODO: Date/version etc. label"
Changed lines of the file:
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@@
 		)
 	)
-	(gr_text "Rowan 1.0 (Prototype 1)\nTom Carlson 2024\nhello@divergentwaves.co.uk"
+	(gr_text "Rowan 1.1 (Production 1)\nTom Carlson 2024-2025\nhello@divergentwaves.co.uk"
 		(at 218.75 133.75 0)
 		(layer "B.SilkS")
@@
 		)
 	)
-	(gr_text "Rowan 1.0 (Prototype 1)\nTom Carlson 2024\nhello@divergentwaves.co.uk"
+	(gr_text "Rowan 1.1 (Production 1)\nTom Carlson 2024-2025\nhello@divergentwaves.co.uk"
 		(at 226 100.5 0)
 		(layer "B.SilkS")
@@
 		)
 	)
-	(gr_text "Rowan 1.0 (Prototype 1)\nTom Carlson 2024\nhello@divergentwaves.co.uk"
+	(gr_text "Rowan 1.1 (Production 1)\nTom Carlson 2024-2025\nhello@divergentwaves.co.uk"
 		(at 147.5 143.25 0)
 		(layer "B.SilkS")
@@
 		)
 	)
-	(gr_text "Bottom board to top board:\nTrig A\nTrig B\nEarth\n\nUnquant A\nChro A\nEarth\n\nUnquant B\nChro B\nEarth\n\nLED driver\n+5v\nEarth\n\n\n"
-		(at 247.1 128.6 0)
-		(layer "Cmts.User")
-		(effects
-			(font
-				(size 1.5 1.5)
-				(thickness 0.3)
-				(bold yes)
-			)
-			(justify left bottom)
-		)
-	)
 	(gr_text "Horizontal center"
 		(at 201.8 146.6 0)
@@
 		(layer "Cmts.User")
 		(effects
-			(font
-				(size 1.5 1.5)
-				(thickness 0.3)
-				(bold yes)
-			)
-			(justify left bottom)
-		)
-	)
-	(gr_text "TODO:\nDate/version etc. label"
-		(at 180.25 153.5 0)
-		(layer "Cmts.User")
-		(effects
-			(font
-				(size 1 1)
-				(thickness 0.15)
-			)
-			(justify left bottom)
-		)
-	)
-	(gr_text "LED centerline (Top)"
-		(at 246.4 129.2488 0)
-		(layer "Cmts.User")
-		(effects
