File: oneshot/oneshot.kicad_sch (KiCad schematic)
At the start: 52 parts, among them J11 Conn_02x05_Odd_Even, J16 Conn_01x02 (3u), J2 Conn_01x04, J25 Conn_01x04, J26 Conn_01x04, J27 Conn_01x04, J3 Conn_01x04, J4 Conn_01x04, J6 Conn_01x04, J7 Conn_01x04, J8 Conn_01x04, Q1 MMBT3904, U1 TL072, U2 TL072, U3 ONESHOT, U4 TL072, U5 LM1117DT-5.0

Commit message: Updating oneshot project files
These are for the 1.1 (Prototype 2) PCBs
Parts:
- J16: footprint Connector_PinHeader_2.54mm:PinHeader_1x02_P2.54mm_Vertical -> Connector_JST:JST_XH_B2B-XH-A_1x02_P2.50mm_Vertical
Changed lines of the file:
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@@
 			)
 		)
-		(property "Footprint" "Connector_PinHeader_2.54mm:PinHeader_1x02_P2.54mm_Vertical"
+		(property "Footprint" "Connector_JST:JST_XH_B2B-XH-A_1x02_P2.50mm_Vertical"
 			(at 246.38 153.67 0)
 			(effects
